File: Materiel/PCB/CarteInterface/PCBProjet.kicad_pcb (KiCad board)
At the start: 2 copper layers, 65 x 56 mm, 21 parts

Commit message: Travailler sur manuel technique
Other:
- net class Default removed
